Commit message: 221125 Add ODOM

File: rudolph_description/urdf/rudolph.urdf.xacro (robot description, xacro)
@@ -1,186 +1,162 @@
-<?xml version="1.0"?>
-    <robot xmlns:xacro="http://www.ros.org/wiki/xacro" name="mobile_robot">
-    <link name="base_footprint"/>
-    <joint name="base_joint" type="fixed">
-        <parent link="base_footprint"/>
-        <child link="base_link" />
-        <origin xyz="0 0.0 0.07" rpy="0 0 0.0"/>
-    </joint>
-    <link name="base_link">
-        <visual>
-            <geometry>
-                <box size="2 1 0.7"/>
-            </geometry>
-        </visual>
-        <collision>
-            <geometry>
-                <box size="2 1 0.7"/>
-            </geometry>
-        </collision>
-        <inertial>
-          <mass value="4"/>
-          <inertia ixx="0.4967" ixy="0.0" ixz="0" iyy="1.4967" iyz="0" izz="1.6667"/>
-        </inertial>
-    </link>
-<!--............................................rf_wheel...................................................... -->
-    <link name= "rf_wheel">
-        <visual>
-	        <origin rpy="1.570795 0 0" xyz="0 0 0"/>
-	        <geometry>
-	            <cylinder length="0.2" radius="0.5"/>
-	        </geometry>
-        </visual>
-        <collision>
-	        <origin rpy="1.570795 0 0" xyz="0 0 0"/>
-	            <geometry>
-	                <cylinder length="0.2" radius="0.5"/>
-	            </geometry>
-        </collision>
-        <inertial>
-	        <origin rpy="1.570795 0 0" xyz="0 0 0"/>
-            <mass value="1"/>
-            <inertia ixx="0.06583" ixy="0.0" ixz="0.0" iyy="0.06583" iyz="0.0" izz="0.125"/>
-        </inertial>
-    </link>
-    <joint name="body_rf_wheel" type="continuous">
-        <axis xyz="0 1 0"/>
-        <parent link="base_link"/>
-        <child link="rf_wheel"/>
-        <origin rpy="0 0 0" xyz="0.7 -0.6 0"/>
-        <limit effort="100" velocity="1.0"/>
-    </joint>
-<!--............................................rb_wheel...................................................... -->
-    <link name= "rb_wheel">
-        <visual>
-	        <origin rpy="1.570795 0 0" xyz="0 0 0"/>
-	        <geometry>
-	            <cylinder length="0.2" radius="0.5"/>
-	        </geometry>
-        </visual>
-        <collision>
-	        <origin rpy="1.570795 0 0" xyz="0 0 0"/>
-	        <geometry>
-	            <cylinder length="0.2" radius="0.5"/>
-	        </geometry>
-        </collision>
-        <inertial>
-	        <origin rpy="1.570795 0 0" xyz="0 0 0"/>
-            <mass value="1"/>
-            <inertia ixx="0.06583" ixy="0.0" ixz="0.0" iyy="0.06583" iyz="0.0" izz="0.125"/>
-        </inertial>
-    </link>
-    <joint name="body_rb_wheel" type="continuous">
-        <axis xyz="0 1 0"/>
-        <parent link="base_link"/>
-        <child link="rb_wheel"/>
-        <origin rpy="0 0 0" xyz="-0.7 -0.6 0"/>
-        <limit effort="100" velocity="1.0"/>
-    </joint>
-<!--............................................lf_wheel...................................................... -->
-    <link name= "lf_wheel">
-        <visual>
-	        <origin rpy="1.570795 0 0" xyz="0 0 0"/>
-	        <geometry>
-	            <cylinder length="0.2" radius="0.5"/>
-	        </geometry>
-        </visual>
-        <collision>
-	        <origin rpy="1.570795 0 0" xyz="0 0 0"/>
-	        <geometry>
-	            <cylinder length="0.2" radius="0.5"/>
-	        </geometry>
-        </collision>
-        <inertial>
-	        <origin rpy="1.570795 0 0" xyz="0 0 0"/>
-            <mass value="1"/>
-            <inertia ixx="0.06583" ixy="0.0" ixz="0.0" iyy="0.06583" iyz="0.0" izz="0.125"/>
-        </inertial>
-    </link>
-    <joint name="body_lf_wheel" type="continuous">
-        <axis xyz="0 1 0"/>
-        <parent link="base_link"/>
-        <child link="lf_wheel"/>
-        <origin rpy="0 0 0" xyz="0.7 0.6 0"/>
-        <limit effort="100" velocity="1.0"/>
-    </joint>
-<!--............................................lb_wheel...................................................... -->
-    <link name= "lb_wheel">
-        <visual>
-	        <origin rpy="1.570795 0 0" xyz="0 0 0"/>
-	        <geometry>
-	            <cylinder length="0.2" radius="0.5"/>
-	        </geometry>
-        </visual>
-        <collision>
-	        <origin rpy="1.570795 0 0" xyz="0 0 0"/>
-	        <geometry>
-	            <cylinder length="0.2" radius="0.5"/>
-	        </geometry>
-        </collision>
-        <inertial>
-	        <origin rpy="1.570795 0 0" xyz="0 0 0"/>
-            <mass value="1"/>
-            <inertia ixx="0.06583" ixy="0.0" ixz="0.0" iyy="0.06583" iyz="0.0" izz="0.125"/>
-        </inertial>
-    </link>
-    <joint name="body_lb_wheel" type="continuous">
-        <axis xyz="0 1 0"/>
-        <parent link="base_link"/>
-        <child link="lb_wheel"/>
-        <origin rpy="0 0 0" xyz="-0.7 0.6 0"/>
-        <limit effort="100" velocity="1.0"/>
-    </joint>
-<!--............................................trnasmission...................................................... -->
-    <transmission name="rf_transmission">
-        <type>transmission_interface/SimpleTransmission</type>
-        <actuator name="rf_motor">
-            <mechanicalReduction>1</mechanicalReduction>
-        </actuator>
-        <joint name="body_rf_wheel">
-            <hardwareInterface>hardware_interface/PositionJointInterface</hardwareInterface>
-        </joint>
-    </transmission>
-    <transmission name="rb_transmission">
-        <type>transmission_interface/SimpleTransmission</type>
-        <actuator name="rb_motor">
-            <mechanicalReduction>1</mechanicalReduction>
-        </actuator>
-        <joint name="body_rb_wheel">
-            <hardwareInterface>hardware_interface/PositionJointInterface</hardwareInterface>
-        </joint>
-    </transmission>
-    <transmission name="lf_transmission">
-        <type>transmission_interface/SimpleTransmission</type>
-        <actuator name="lf_motor">
-            <mechanicalReduction>1</mechanicalReduction>
-        </actuator>
-        <joint name="body_lf_wheel">
-            <hardwareInterface>hardware_interface/PositionJointInterface</hardwareInterface>
-        </joint>
-    </transmission>
-    <transmission name="lb_transmission">
-        <type>transmission_interface/SimpleTransmission</type>
-        <actuator name="lb_motor">
-            <mechanicalReduction>1</mechanicalReduction>
-        </actuator>
-        <joint name="body_lb_wheel">
-            <hardwareInterface>hardware_interface/PositionJointInterface</hardwareInterface>
-        </joint>
-    </transmission>
-    <gazebo>
-        <plugin name="skid_steer_drive_controller" filename="libgazebo_ros_skid_steer_drive.so">
-   	        <updateRate>100.0</updateRate>
-   	        <robotNamespace>/</robotNamespace>
-   	        <leftFrontJoint>body_lf_wheel</leftFrontJoint>
-   	        <rightFrontJoint>body_rf_wheel</rightFrontJoint>
-   	        <leftRearJoint>body_lb_wheel</leftRearJoint>
-   	        <rightRearJoint>body_rb_wheel</rightRearJoint>
-  	        <wheelSeparation>0.2</wheelSeparation>
-  	        <wheelDiameter>0.4</wheelDiameter>
-	        <torque>100</torque>
-  	        <robotBaseFrame>body</robotBaseFrame>
-  	        <topicName>cmd_vel</topicName>
-  	        <broadcastTF>false</broadcastTF>
-  	    </plugin>
-    </gazebo>
+<?xml version="1.0" ?>
+<robot name="rudolph" xmlns:xacro="http://ros.org/wiki/xacro">
+  <xacro:include filename="$(find rudolph_description)/urdf/common_properties.xacro"/>
+  <xacro:include filename="$(find rudolph_description)/urdf/rudolph.gazebo.xacro"/>
+  <link name="base_footprint"/>
+  <joint name="base_joint" type="fixed">
+    <parent link="base_footprint"/>
+    <child link="base_link"/>
+    <origin xyz="0.0 0.0 0.010" rpy="0 0 0"/>
+  </joint>
+  <link name="base_link">
+    <visual>
+      <origin xyz="0 0 0.098" rpy="1.57 0 1.57"/>
+      <geometry>
+        <mesh filename="package://rudolph_description/meshes/bases/body1.stl" scale="0.001 0.001 0.001"/>
+      </geometry>
+      <material name="light_black"/>
+    </visual>
+    <collision>
+      <origin xyz="0 0 0.098" rpy="0 0 0"/>
+      <geometry>
+        <box size="0.1 0.395 0.1"/>
+      </geometry>
+    </collision>
+    <inertial>
+      <origin xyz="0 0 0" rpy="0 0 0"/>
+      <mass value="8.2573504e-01"/>
+      <inertia ixx="2.2124416e-03" ixy="-1.2294101e-05" ixz="3.4938785e-05"
+               iyy="2.1193702e-03" iyz="-5.0120904e-06"
+               izz="2.0064271e-03" />
+    </inertial>
+  </link>
+  <joint name="wheel_left_joint" type="continuous">
+    <parent link="base_link"/>
+    <child link="wheel_left_link"/>
+    <origin xyz="0.0 0.08 0.023" rpy="-1.57 0 0"/>
+    <axis xyz="0 0 1"/>
+  </joint>
+  <link name="wheel_left_link">
+    <visual>
+      <origin xyz="0.105 -0.0265 0.13" rpy="0 1.57 0"/>
+      <geometry>
+        <mesh filename="package://rudolph_description/meshes/wheels/wheel.stl" scale="0.001 0.001 0.001"/>
+      </geometry>
+      <material name="dark"/>
+    </visual>
+    <collision>
+      <origin xyz="0 0 0" rpy="0 0 0"/>
+      <geometry>
+        <cylinder length="0.018" radius="0.033"/>
+      </geometry>
+    </collision>
+    <inertial>
+      <origin xyz="0 0 0" />
+      <mass value="2.8498940e-02" />
+      <inertia ixx="1.1175580e-05" ixy="-4.2369783e-11" ixz="-5.9381719e-09"
+               iyy="1.1192413e-05" iyz="-1.4400107e-11"
+               izz="2.0712558e-05" />
+      </inertial>
+  </link>
+  <joint name="wheel_right_joint" type="continuous">
+    <parent link="base_link"/>
+    <child link="wheel_right_link"/>
+    <origin xyz="0.0 -0.080 0.023" rpy="-1.57 0 0"/>
+    <axis xyz="0 0 1"/>
+  </joint>
+  <link name="wheel_right_link">
+    <visual>
+      <origin xyz="0.105 -0.0265 -0.13" rpy="0 1.57 0"/>
+      <geometry>
+        <mesh filename="package://rudolph_description/meshes/wheels/wheel.stl" scale="0.001 0.001 0.001"/>
+      </geometry>
+      <material name="dark"/>
+    </visual>
+    <collision>
+      <origin xyz="0 0 0" rpy="0 0 0"/>
+      <geometry>
+        <cylinder length="0.018" radius="0.033"/>
+      </geometry>
+    </collision>
+    <inertial>
+      <origin xyz="0 0 0" />
+      <mass value="2.8498940e-02" />
+      <inertia ixx="1.1175580e-05" ixy="-4.2369783e-11" ixz="-5.9381719e-09"
+               iyy="1.1192413e-05" iyz="-1.4400107e-11"
+               izz="2.0712558e-05" />
+      </inertial>
+  </link>
+  <joint name="caster_back_joint" type="fixed">
+    <parent link="base_link"/>
+    <child link="caster_back_link"/>
+    <origin xyz="-0.081 0 -0.004" rpy="-1.57 0 0"/>
+  </joint>
+  <link name="caster_back_link">
+    <collision>
+      <origin xyz="0 0.001 0" rpy="0 0 0"/>
+      <geometry>
+        <box size="0.030 0.009 0.020"/>
+      </geometry>
+    </collision>
+    <inertial>
+      <origin xyz="0 0 0" />
+      <mass value="0.005" />
+      <inertia ixx="0.001" ixy="0.0" ixz="0.0"
+               iyy="0.001" iyz="0.0"
+               izz="0.001" />
+    </inertial>
+  </link>
+  <joint name="imu_joint" type="fixed">
+    <parent link="base_link"/>
+    <child link="imu_link"/>
+    <origin xyz="-0.032 0 0.068" rpy="0 0 0"/>
+  </joint>
+  <link name="imu_link"/>
+  <joint name="scan_joint" type="fixed">
+    <parent link="base_link"/>
+    <child link="base_scan"/>
+    <origin xyz="-0.032 0 0.172" rpy="0 0 0"/>
+  </joint>
+  <link name="base_scan">
+    <visual>
+      <origin xyz="0 0 0.24" rpy="0 0 1.57"/>
+      <geometry>
+        <mesh filename="package://rudolph_description/meshes/sensors/lds(original).stl" scale="0.001 0.001 0.001"/>
+      </geometry>
+      <material name="dark"/>
+    </visual>
+    <collision>
+      <origin xyz="0.015 0 -0.0065" rpy="0 0 0"/>
+      <geometry>
+        <cylinder length="0.0315" radius="0.055"/>
+      </geometry>
+    </collision>
+    <inertial>
+      <mass value="0.114" />
+      <origin xyz="0 0 0" />
+      <inertia ixx="0.001" ixy="0.0" ixz="0.0"
+               iyy="0.001" iyz="0.0"
+               izz="0.001" />
+    </inertial>
+  </link>
+  <joint name="camera_joint" type="fixed">
+    <origin xyz="-0.032 0.0 0.172" rpy="0 0 0"/>
+    <parent link="base_link"/>
+    <child link="camera_link"/>
+  </joint>
+  <link name="camera_link">
+    <visual>
+      <origin xyz="0.23 0 0.2" rpy="1.57 0.0 -1.57"/>
+      <geometry>
+        <mesh filename="package://rudolph_description/meshes/sensors/omo_r1_camera.stl" scale="0.001 0.001 0.001"/>
+      </geometry>
+      <material name="dark"/>
+    </visual>
+    <collision>
+      <origin xyz="0 0 0.0" rpy="0 0.0 0"/>
+      <geometry>
+        <mesh filename="package://rudolph_description/meshes/sensors/omo_r1_camera.stl" scale="0.001 0.001 0.001"/>
+      </geometry>
+    </collision>
+  </link>
 </robot>

Commit message: 1208

File: rudolph_description/urdf/rudolph.urdf.xacro (robot description, xacro)
@@ -4,12 +4,50 @@
      For more information, please see http://wiki.ros.org/sw_urdf_exporter -->
 <robot
-  name="rudolph_urdf">
-  <link
-    name="base_footprint"/>
+  name="rudolph_description">
+  <link
+    name="base_footprint">
+    <inertial>
+      <origin
+        xyz="0.0689100280019426 0.00900000000230574 0.0761077688742865"
+        rpy="0 0 0" />
+      <mass
+        value="0.00777136970807385" />
+      <inertia
+        ixx="3.52976794817517E-07"
+        ixy="4.01095779280605E-23"
+        ixz="1.20969262982029E-09"
+        iyy="6.78327211008114E-07"
+        iyz="7.16782676416494E-21"
+        izz="6.78004492386885E-07" />
+    </inertial>
+    <visual>
+      <origin
+        xyz="0 0 0"
+        rpy="0 0 0" />
+      <geometry>
+        <mesh
+          filename="package://rudolph_description/meshes/base_footprint.STL" />
+      </geometry>
+      <material
+        name="">
+        <color
+          rgba="0.792156862745098 0.819607843137255 0.933333333333333 1" />
+      </material>
+    </visual>
+    <collision>
+      <origin
+        xyz="0 0 0"
+        rpy="0 0 0" />
+      <geometry>
+        <mesh
+          filename="package://rudolph_description/meshes/base_footprint.STL" />
+      </geometry>
+    </collision>
+  </link>
   <link
     name="base_link">
     <inertial>
       <origin
-        xyz="-0.198744010402315 0.000174583761450766 0.143169546471357"
+        xyz="-0.198744010402315 0.000174583761450815 0.143169546471357"
         rpy="0 0 0" />
       <mass
@@ -20,5 +58,5 @@
         ixz="3.76767258085507E-05"
         iyy="0.322483556824621"
-        iyz="-3.3367514082637E-06"
+        iyz="-3.33675140826365E-06"
         izz="0.34473391633269" />
     </inertial>
@@ -51,5 +89,5 @@
     type="fixed">
     <origin
-      xyz="0.31976 0 -0.0431"
+      xyz="0 0 0.055"
       rpy="0 0 0" />
     <parent
@@ -64,15 +102,15 @@
     <inertial>
       <origin
-        xyz="5.62079272015126E-10 7.35240311688923E-09 -0.00280091246570427"
-        rpy="0 0 0" />
-      <mass
-        value="0.16892790393776" />
-      <inertia
-        ixx="0.000180293267647714"
-        ixy="3.4968846919059E-10"
-        ixz="-5.92226218447572E-13"
-        iyy="0.0001802932498828"
-        iyz="-1.35428150724921E-11"
-        izz="0.000340883721564796" />
+        xyz="5.65954616504882E-10 7.36872513007469E-09 -0.00280091247127531"
+        rpy="0 0 0" />
+      <mass
+        value="0.168927903786118" />
+      <inertia
+        ixx="0.000180293267616765"
+        ixy="3.49702912743621E-10"
+        ixz="-5.96562390165147E-13"
+        iyy="0.000180293249897517"
+        iyz="-1.35611495762941E-11"
+        izz="0.000340883721561127" />
     </inertial>
     <visual>
@@ -104,6 +142,6 @@
     type="continuous">
     <origin
-      xyz="0.00024307 0.2084 0.00010011"
-      rpy="-1.5708 0 0" />
+      xyz="0.000243065284555088 0.208400000002307 0.000100106132487177"
+      rpy="-1.5707963267949 0 0" />
     <parent
       link="base_link" />
@@ -117,15 +155,15 @@
     <inertial>
       <origin
-        xyz="5.6243787405208E-10 -7.35308421095926E-09 0.00280091246576517"
-        rpy="0 0 0" />
-      <mass
-        value="0.168927903936188" />
-      <inertia
-        ixx="0.000180293267644942"
-        ixy="-3.49688656954827E-10"
-        ixz="5.9278420728745E-13"
-        iyy="0.000180293249883525"
-        iyz="-1.35438613193214E-11"
-        izz="0.000340883721562999" />
+        xyz="5.66313440586441E-10 -7.36940622414473E-09 0.00280091247133624"
+        rpy="0 0 0" />
+      <mass
+        value="0.168927903784547" />
+      <inertia
+        ixx="0.000180293267613993"
+        ixy="-3.49703100507898E-10"
+        ixz="5.9712037933952E-13"
+        iyy="0.000180293249898242"
+        iyz="-1.35621958235081E-11"
+        izz="0.00034088372155933" />
     </inertial>
     <visual>
@@ -157,6 +195,6 @@
     type="continuous">
     <origin
-      xyz="0.00024307 -0.2084 0.00010011"
-      rpy="-1.5708 0 0" />
+      xyz="0.000243065284555311 -0.208399999997693 0.000100106132487593"
+      rpy="-1.5707963267949 0 0" />
     <parent
       link="base_link" />
@@ -176,8 +214,8 @@
       <inertia
         ixx="0.000181440969274869"
-        ixy="3.79381726757463E-05"
-        ixz="-4.39393075157974E-11"
-        iyy="0.000117632047892803"
-        iyz="2.10111827244022E-12"
+        ixy="3.79381726757464E-05"
+        ixz="-4.39393075162352E-11"
+        iyy="0.000117632047892804"
+        iyz="2.10111827256733E-12"
         izz="0.000234531410256484" />
     </inertial>
@@ -210,10 +248,63 @@
     type="fixed">
     <origin
-      xyz="-0.52941 0 -0.022461"
-      rpy="-1.5708 0 0" />
+      xyz="-0.529406195960553 0 -0.0224614324940508"
+      rpy="-1.5707963267949 0 0" />
     <parent
       link="base_link" />
     <child
       link="caster_back_link" />
+    <axis
+      xyz="0 0 0" />
+  </joint>
+  <link
+    name="camera_link">
+    <inertial>
+      <origin
+        xyz="0.00593852099290992 5.09399578095537E-07 0.00784055172380349"
+        rpy="0 0 0" />
+      <mass
+        value="0.0581895549431422" />
+      <inertia
+        ixx="2.149536557957E-05"
+        ixy="-4.25271059883761E-10"
+        ixz="-4.30001305453024E-08"
+        iyy="7.2478764849786E-06"
+        iyz="3.06968376267156E-10"
+        izz="2.484439535279E-05" />
+    </inertial>
+    <visual>
+      <origin
+        xyz="0 0 0"
+        rpy="0 0 0" />
+      <geometry>
+        <mesh
+          filename="package://rudolph_description/meshes/camera_link.STL" />
+      </geometry>
+      <material
+        name="">
+        <color
+          rgba="0.23921568627451 0.23921568627451 0.235294117647059 1" />
+      </material>
+    </visual>
+    <collision>
+      <origin
+        xyz="0 0 0"
+        rpy="0 0 0" />
+      <geometry>
+        <mesh
+          filename="package://rudolph_description/meshes/camera_link.STL" />
+      </geometry>
+    </collision>
+  </link>
+  <joint
+    name="camera_joint"
+    type="fixed">
+    <origin
+      xyz="0.0537459832126193 0.000590752056278902 0.348100106132424"
+      rpy="0 0 0" />
+    <parent
+      link="base_link" />
+    <child
+      link="camera_link" />
     <axis
       xyz="0 0 0" />
@@ -263,5 +354,5 @@
     type="fixed">
     <origin
-      xyz="-0.027357 0 0.3851"
+      xyz="-0.0273569347154501 0 0.385100106132424"
       rpy="0 0 0" />
     <parent
@@ -269,57 +360,4 @@
     <child
       link="base_scan" />
-    <axis
-      xyz="0 0 0" />
-  </joint>
-  <link
-    name="camera_link">
-    <inertial>
-      <origin
-        xyz="0.00593852099291015 5.09399578095537E-07 0.00784055172380355"
-        rpy="0 0 0" />
-      <mass
-        value="0.0581895549431422" />
-      <inertia
-        ixx="2.149536557957E-05"
-        ixy="-4.25271059883842E-10"
-        ixz="-4.30001305453022E-08"
-        iyy="7.2478764849786E-06"
-        iyz="3.06968376267082E-10"
-        izz="2.484439535279E-05" />
-    </inertial>
-    <visual>
-      <origin
-        xyz="0 0 0"
-        rpy="0 0 0" />
-      <geometry>
-        <mesh
-          filename="package://rudolph_description/meshes/camera_link.STL" />
-      </geometry>
-      <material
-        name="">
-        <color
-          rgba="0.23921568627451 0.23921568627451 0.235294117647059 1" />
-      </material>
-    </visual>
-    <collision>
-      <origin
-        xyz="0 0 0"
-        rpy="0 0 0" />
-      <geometry>
-        <mesh
-          filename="package://rudolph_description/meshes/camera_link.STL" />
-      </geometry>
-    </collision>
-  </link>
-  <joint
-    name="camera_joint"
-    type="fixed">
-    <origin
-      xyz="0.053746 0.00059075 0.3481"
-      rpy="0 0 0" />
-    <parent
-      link="base_link" />
-    <child
-      link="camera_link" />
     <axis
       xyz="0 0 0" />
